File: Preamp board.kicad_pcb (KiCad board)
At the start: 2 copper layers, 19.1 x 59.6 mm, 23 parts, among them J1 Coil, J2 Rx, J3 DC, J4 DC, U1 Preamp

Commit message: Updated version number on pcb to v1.0
Other:
- board text added: "04/2020 v1.0"
- board text removed: "04/2020 v0.3"

Commit message: Updated version date
Other:
- board text added: "11/2021 v1.0"
- board text removed: "04/2020 v1.0"
Changed lines of the file:
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@@
       (effects (font (size 0.75 0.75) (thickness 0.15)))
     )
-    (pad 2 smd roundrect (at 2.1375 0 180) (size 1.125 3.4) (layers F.Cu F.Paste F.Mask) (roundrect_rratio 0.2222204444444444)
+    (pad 2 smd roundrect (at 2.1375 0 180) (size 1.125 3.4) (layers F.Cu F.Paste F.Mask) (roundrect_rratio 0.2222195555555556)
       (net 5 "Net-(L1-Pad1)"))
-    (pad 1 smd roundrect (at -2.1375 0 180) (size 1.125 3.4) (layers F.Cu F.Paste F.Mask) (roundrect_rratio 0.2222204444444444)
+    (pad 1 smd roundrect (at -2.1375 0 180) (size 1.125 3.4) (layers F.Cu F.Paste F.Mask) (roundrect_rratio 0.2222195555555556)
       (net 2 "Net-(C1-Pad1)"))
     (model ${KISYS3DMOD}/Inductor_SMD.3dshapes/L_1812_4532Metric.wrl
@@
       (effects (font (size 0.75 0.75) (thickness 0.15)))
     )
-    (pad 2 smd roundrect (at 2.1375 0 90) (size 1.125 3.4) (layers F.Cu F.Paste F.Mask) (roundrect_rratio 0.2222204444444444)
+    (pad 2 smd roundrect (at 2.1375 0 90) (size 1.125 3.4) (layers F.Cu F.Paste F.Mask) (roundrect_rratio 0.2222195555555556)
       (net 8 "Net-(C2-Pad2)"))
-    (pad 1 smd roundrect (at -2.1375 0 90) (size 1.125 3.4) (layers F.Cu F.Paste F.Mask) (roundrect_rratio 0.2222204444444444)
+    (pad 1 smd roundrect (at -2.1375 0 90) (size 1.125 3.4) (layers F.Cu F.Paste F.Mask) (roundrect_rratio 0.2222195555555556)
       (net 5 "Net-(L1-Pad1)"))
     (model ${KISYS3DMOD}/Inductor_SMD.3dshapes/L_1812_4532Metric.wrl
@@
     (effects (font (size 1.5 1.5) (thickness 0.3)) (justify mirror))
   )
-  (gr_text "04/2020\nv1.0" (at 65.28 129.74 -90) (layer B.SilkS)
+  (gr_text "11/2021\nv1.0" (at 65.28 129.74 -90) (layer B.SilkS)
     (effects (font (size 1 1) (thickness 0.25)) (justify left mirror))
   )
